File: hardware/proof/gate-proof/gate-proof.kicad_pcb (KiCad board)
At the start: 2 copper layers, 60 x 20 mm, 4 parts, among them J1 MAINS_IN, J2 LV_IN

Commit message: feat(board-check): measure the workmanship rules and require KiCad's in every rules file [SOL-BOARD-LAYOUT-WORKMANSHIP-ITEMS.C2]
The pre-order check now requires a track_angle and a track_segment_length
rule on every track in each design's rules file, and measures from the
layout what KiCad does not: stubs, route length against the shortest
straight-line tree of the net's pads, track direction against the board's
edges, entry into long pads, and narrowing below the net class's width away
from a pad. Each figure is a project text variable, missing or malformed
figures fail by name, and the report states each figure it read. The pad
geometry and the tree live once in board_geometry, which the views and the
locked-copper check now share. The gate's proof design is tidied to 45-degree
corners and carries the rules, and each new rule has a seeded fault.

Co-Authored-By: Claude Opus 5.5 (1M context) <noreply@anthropic.com>
Routing:
- net /MAINS_N: track 17.7 -> 16.2 mm
- net /LV_B: track 17.7 -> 16.2 mm
Changed lines of the file:
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@@
 		)
 	)
+	(property "MAINS" "present")
+	(property "NOT_FOR_MANUFACTURE" "true")
 	(footprint "proof:PinHeader_1x02_P2.54mm_Vertical"
 		(layer "F.Cu")
@@
 	)
 	(segment
-		(start 25.16 12.54)
+		(start 22.62 12.54)
 		(end 25.16 10)
 		(width 0.5)
@@
 	(segment
 		(start 10 12.54)
-		(end 25.16 12.54)
+		(end 22.62 12.54)
 		(width 0.5)
 		(layer "F.Cu")
@@
 	)
 	(segment
-		(start 55.16 12.54)
+		(start 40 12.54)
+		(end 52.62 12.54)
+		(width 0.25)
+		(layer "F.Cu")
+		(net "/LV_B")
+	)
+	(segment
+		(start 52.62 12.54)
 		(end 55.16 10)
 		(width 0.25)
 		(layer "F.Cu")
-		(net "/LV_B")
-	)
-	(segment
-		(start 40 12.54)
-		(end 55.16 12.54)
-		(width 0.25)
-		(layer "F.Cu")

Commit message: feat(hardware): check a board's connectivity against its pin allocation record, each fault proven on a throwaway design [SOL-HW-CONNECTIVITY-CHECK.C1, .C2, .C3, .C4, .C5]
Co-Authored-By: Claude Sonnet 5.5 <noreply@anthropic.com>
Parts:
- added U1: CTRL, proof:Controller_1x02, F.Cu at (43.0, 10.0)
Changed lines of the file:
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@@
 	(property "MAINS" "present")
 	(property "NOT_FOR_MANUFACTURE" "true")
+	(footprint "proof:Controller_1x02"
+		(layer "F.Cu")
+		(at 43 10)
+		(descr "Controller-style part with two port pins, for the proof design")
+		(tags "proof controller")
+		(property "Reference" "U1"
+			(at 0 -2.38 0)
+			(layer "F.Fab")
+			(effects
+				(font
+					(size 1 1)
+					(thickness 0.15)
+				)
+			)
+		)
+		(property "Value" "CTRL"
+			(at 0 4.92 0)
+			(layer "F.Fab")
+			(effects
+				(font
+					(size 1 1)
+					(thickness 0.15)
+				)
+			)
+		)
+		(property "Datasheet" ""
+			(at 0 0 0)
+			(layer "F.Fab")
+			(hide yes)
+			(effects
+				(font
+					(size 1.27 1.27)
+				)
+			)
+		)
+		(property "Description" ""
+			(at 0 0 0)
+			(layer "F.Fab")
+			(hide yes)
+			(effects
+				(font
+					(size 1.27 1.27)
+				)
+			)
+		)
+		(sheetname "/")
+		(sheetfile "gate-proof.kicad_sch")
+		(attr through_hole)
+		(duplicate_pad_numbers_are_jumpers no)
+		(fp_rect
+			(start -0.9 -0.9)
+			(end 0.9 3.44)
+			(stroke
+				(width 0.05)
+				(type solid)
+			)
+			(fill no)
+			(layer "F.CrtYd")
+		)
+		(pad "1" thru_hole rect
+			(at 0 0)
+			(size 1.7 1.7)
+			(drill 1)
+			(layers "*.Cu" "*.Mask")
+			(remove_unused_layers no)
+			(net "/LV_A")
+		)
+		(pad "2" thru_hole circle
+			(at 0 2.54)
+			(size 1.7 1.7)
+			(drill 1)
+			(layers "*.Cu" "*.Mask")
+			(remove_unused_layers no)
+			(net "/LV_B")
+		)
+		(embedded_fonts no)
+	)
 	(footprint "proof:PinHeader_1x02_P2.54mm_Vertical"
 		(layer "F.Cu")
