File: hardware/proof/method-proof/method-proof.kicad_pcb (KiCad board)
At the start: 4 copper layers, 40 x 30 mm, 21 parts, among them J1 5V_IN, J2 OUT, J3 PA1, U1 MCP1700T-3302E/TT, U2 MSPS003F4SPW20R

Commit message: hardware(method-proof): the +5V tap to R1's feed moved from between C1 and U1's input pin to the JP1 branch of the pour, relocked (layout-review.md, round 1, finding 1.2)
Co-Authored-By: Claude Sonnet 5.5 <noreply@anthropic.com>
Routing:
- net +5V: track 33.5 -> 34.8 mm
Changed lines of the file:
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@@
 	)
 	(via
-		(at 113.6 109.5)
+		(at 113 107.9)
 		(size 0.6)
 		(drill 0.2)
@@
 	)
 	(segment
-		(start 113.6 109.5)
-		(end 117.66 109.5)
+		(start 116.06 107.9)
+		(end 118.66 110.5)
 		(width 0.5)
 		(locked yes)
@@
 	)
 	(segment
-		(start 117.66 109.5)
-		(end 118.66 110.5)
+		(start 113 107.9)
+		(end 116.06 107.9)
 		(width 0.5)
 		(locked yes)

Commit message: hardware(method-proof): a second ground via of its own beside each of C1's, C2's and C3's ground pads, relocked (layout-review.md, round 1, finding 1.3)
Co-Authored-By: Claude Sonnet 5.5 <noreply@anthropic.com>
Routing:
- net GND: vias 11 -> 14
Changed lines of the file:
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@@
+	)
+	(via
+		(at 113.3 112.54)
+		(size 0.6)
+		(drill 0.2)
+		(layers "F.Cu" "B.Cu")
+		(locked yes)
+		(net "GND")
 	)
 	(via
@@
 	)
 	(via
+		(at 119.55 112.62)
+		(size 0.6)
+		(drill 0.2)
+		(layers "F.Cu" "B.Cu")
+		(locked yes)
+		(net "GND")
+	)
+	(via
 		(at 106.7 106.5)
 		(size 0.6)
 		(drill 0.2)
+		(layers "F.Cu" "B.Cu")
+		(locked yes)
+		(net "GND")
+	)
+	(via
+		(at 117.8 102.46)
+		(size 0.6)
+		(drill 0.2)

Commit message: hardware(method-proof): two ground vias of their own beside each of C4's and C5's ground pads, relocked (layout-review.md, round 1, finding 1.6)
Co-Authored-By: Claude Sonnet 5.5 <noreply@anthropic.com>
Routing:
- net GND: vias 14 -> 18
Changed lines of the file:
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@@
+	)
+	(via
+		(at 110.77 115.5)
+		(size 0.6)
+		(drill 0.2)
+		(layers "F.Cu" "B.Cu")
+		(locked yes)
+		(net "GND")
 	)
 	(via
 		(at 105.5 106.5)
+		(size 0.6)
+		(drill 0.2)
+		(layers "F.Cu" "B.Cu")
+		(locked yes)
+		(net "GND")
+	)
+	(via
+		(at 109.47 114.3)
 		(size 0.6)
 		(drill 0.2)
@@
 	)
 	(via
+		(at 110.77 113)
+		(size 0.6)
+		(drill 0.2)
+		(layers "F.Cu" "B.Cu")
+		(locked yes)
+		(net "GND")
+	)
+	(via
 		(at 106.7 106.5)
 		(size 0.6)
 		(drill 0.2)
+		(layers "F.Cu" "B.Cu")
+		(locked yes)
+		(net "GND")
+	)
+	(via
+		(at 108.82 114.37)
+		(size 0.6)
+		(drill 0.2)

Commit message: hardware(method-proof): two ground vias of their own beside U1's ground pad, relocked (layout-review.md, round 1, finding 1.4)
Co-Authored-By: Claude Sonnet 5.5 <noreply@anthropic.com>
Routing:
- net GND: vias 18 -> 20
Changed lines of the file:
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@@
+	)
+	(via
+		(at 115.81 111.1)
+		(size 0.6)
+		(drill 0.2)
+		(layers "F.Cu" "B.Cu")
+		(locked yes)
+		(net "GND")
 	)
 	(via
@@
 		(size 0.6)
 		(drill 0.2)
+		(layers "F.Cu" "B.Cu")
+		(locked yes)
+		(net "GND")
+	)
+	(via
+		(at 116.94 111.75)
+		(size 0.6)
+		(drill 0.2)
