File: hardware/proof/circuit-review-proof/circuit-review-proof.kicad_pcb (KiCad board)
At the start: 4 copper layers, 238 x 132 mm, 54 parts, among them J1 MKDSN_1.5/3-5.08, J2 HEATER, J3 SENSOR_I2C, J4 SWD, J5 SENSE_IN, J6 5V_IN, Q1 BTA16-600B, Q2 BSS138, Q3 BSS138, U2 MOC3023M, U3 MCP1700T-3302E/TT, U4 MSPS003F4SPW20R, U5 TPS3823-33DBVR

Commit message: fix(hardware): give the tracked proof designs the three fiducials a side with surface-mount parts needs [SOL-PRE-ORDER-CHECK-FIDUCIALS-AND-POLARITY-MARKS.C5]
Co-Authored-By: Claude Sonnet 5.5 <noreply@anthropic.com>
Parts:
- added FID1: Fiducial, Fiducial:Fiducial_1mm_Mask2mm, F.Cu at (12.0, 14.0)
- added FID2: Fiducial, Fiducial:Fiducial_1mm_Mask2mm, F.Cu at (12.0, 130.0)
- added FID3: Fiducial, Fiducial:Fiducial_1mm_Mask2mm, F.Cu at (100.0, 130.0)
- added FID4: Fiducial, Fiducial:Fiducial_1mm_Mask2mm, B.Cu at (16.0, 16.0)
- added FID5: Fiducial, Fiducial:Fiducial_1mm_Mask2mm, B.Cu at (16.0, 126.0)
- added FID6: Fiducial, Fiducial:Fiducial_1mm_Mask2mm, B.Cu at (96.0, 126.0)
