File: hardware/proof/review-proof/review-proof.kicad_sch (KiCad schematic)
At the start: 26 parts, among them J1 MAINS, J2 5V_IN, J4 LOAD, U1 VO3526, U2 AMS1117-3.3, U3 MCP6001-OT, U4 ATtiny85-20M, Y1 8MHz

Commit message: fix(hardware): fit a two-pad crystal whose pads face its capacitors, and keep the R3 rule area clear of its track [SOL-BOARD-LAYOUT-WORKMANSHIP-ITEMS.C3, .C4]
Round 4 finding 4.1: the HC49-SD crystal's pads lie 8.5 mm apart and each
must be entered along its length, so no way of turning it both keeps its two
tracks apart (CLOCK-1) and faces each pad to its capacitor (WORK-1). Y1 is
now a 5.0 by 3.2 mm two-pad crystal from KiCad's own library, its schematic
footprint field changed with it, set just beyond C5 and C6 with each pad
facing its capacitor and both tracks 5.7 mm long; it sits 25.1 mm from C2's
body, so no further part comes within CLOCK-3's 25 mm. The footprint is
swapped with KiCad's own scripting on the closed board, keeping its symbol
link and nets, since Konnect cannot change a placed footprint; the tracks
and placement go through Konnect.

Round 4 finding 4.2: the R3 ground return rule area is redrawn to follow
the track's 45-degree run, so the pour stops 0.35 mm or more from the track and 0.275 mm from R3's pad
everywhere rather than 0.077 mm.

The plan, the rules table and the crystal seeds follow.

Co-Authored-By: Claude Opus 5.5 (1M context) <noreply@anthropic.com>
Parts:
- Y1: footprint Crystal:Crystal_SMD_HC49-SD -> Crystal:Crystal_SMD_5032-2Pin_5.0x3.2mm
Changed lines of the file:
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@@
 			)
 		)
-		(property "Footprint" "Crystal:Crystal_SMD_HC49-SD"
+		(property "Footprint" "Crystal:Crystal_SMD_5032-2Pin_5.0x3.2mm"
 			(at 271.78 40.64 0)
 			(hide yes)

Commit message: feat(hardware): check a board's parts against its specification record and the dated catalogue extract, each fault proven on a throwaway design [SOL-HW-PARTS-CHECK.C1, .C2, .C3, .C4, .C5]
Co-Authored-By: Claude Sonnet 5.5 <noreply@anthropic.com>
Parts:
- C1: LCSC (none) -> C9000004; Rating (none) -> 50V
- C2: LCSC (none) -> C9000005; Rating (none) -> 50V
- C3: LCSC (none) -> C9000018; Rating (none) -> 50V
- C4: LCSC (none) -> C9000020; Rating (none) -> 50V
- C5: LCSC (none) -> C9000022; Rating (none) -> 50V
- C6: LCSC (none) -> C9000023; Rating (none) -> 50V
- D1: LCSC (none) -> C9000025
- FB1: LCSC (none) -> C9000017
- J1: LCSC (none) -> C9000001
- J2: LCSC (none) -> C9000003
- J4: LCSC (none) -> C9000006
- R1: LCSC (none) -> C9000007; Rating (none) -> 0.25W
- R2: LCSC (none) -> C9000015; Rating (none) -> 0.25W
- R3: LCSC (none) -> C9000016; Rating (none) -> 0.25W
- R4: LCSC (none) -> C9000024; Rating (none) -> 0.25W
- TP1: LCSC (none) -> C9000008
- TP2: LCSC (none) -> C9000009
- TP3: LCSC (none) -> C9000010
- TP4: LCSC (none) -> C9000011
- TP5: LCSC (none) -> C9000012
- TP6: LCSC (none) -> C9000013
- U1: LCSC (none) -> C9000002
- U2: LCSC (none) -> C9000026
- U3: LCSC (none) -> C9000014
- U4: LCSC (none) -> C9000019
- Y1: LCSC (none) -> C9000021

Commit message: feat(board): the review proof design closes the findings its own review recorded, with the rules that review judged [SOL-BOARD-REVIEW-PROOF-BASELINE-CLEAN.C1, .C2, .C3]
Co-Authored-By: Claude Sonnet 5.5 <noreply@anthropic.com>
Parts:
- added C7, C8: 1uF, Capacitor_SMD:C_0805_2012Metric, symbol Device:C
- added H1, H2, H3: MountingHole, MountingHole:MountingHole_3.2mm_M3, symbol Mechanical:MountingHole
- U4: footprint Package_DFN_QFN:QFN-20-1EP_4x4mm_P0.5mm_EP2.6x2.6mm -> review-proof:QFN-20-1EP_4x4mm_P0.5mm_EP2.6x2.6mm
Connections:
- net +5V: now also C7.1, C8.1
- net GND: now also C7.2, C8.2
- net MAINS_L: now also J1.2 (Pin_2); no longer J1.1 (Pin_1)
- net MAINS_SW: now also J1.1 (Pin_1); no longer J1.2 (Pin_2)

Commit message: fix(hardware): give the tracked proof designs the three fiducials a side with surface-mount parts needs [SOL-PRE-ORDER-CHECK-FIDUCIALS-AND-POLARITY-MARKS.C5]
Co-Authored-By: Claude Sonnet 5.5 <noreply@anthropic.com>
Parts:
- added FID1, FID2, FID3: Fiducial, Fiducial:Fiducial_1mm_Mask2mm, symbol Mechanical:Fiducial
Changed lines of the file:
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@@
+		)
+	)
+	(symbol
+		(lib_id "Mechanical:Fiducial")
+		(at 147.32 149.86 0)
+		(unit 1)
+		(in_bom no)
+		(on_board yes)
+		(dnp no)
+		(property "Reference" "FID1"
+			(at 147.32 144.78 0)
+			(effects
+				(font
+					(size 1.27 1.27)
+				)
+			)
+		)
+		(property "Value" "Fiducial"
+			(at 147.32 146.685 0)
+			(effects
+				(font
+					(size 1.27 1.27)
+				)
+			)
+		)
+		(property "Footprint" "Fiducial:Fiducial_1mm_Mask2mm"
+			(at 147.32 149.86 0)
+			(hide yes)
+			(effects
+				(font
+					(size 1.27 1.27)
+				)
+			)
+		)
+		(property "LCSC" "C9000032"
+			(at 147.32 149.86 0)
+			(hide yes)
+			(effects
+				(font
+					(size 1.27 1.27)
+				)
+			)
+		)
+		(property "Datasheet" ""
+			(at 147.32 149.86 0)
+			(hide yes)
+			(effects
+				(font
+					(size 1.27 1.27)
+				)
+			)
+		)
+		(property "Description" "Fiducial Marker"
+			(at 147.32 149.86 0)
+			(hide yes)
+			(effects
+				(font
+					(size 1.27 1.27)
+				)
+			)
+		)
+		(instances
+			(project "review-proof"
+				(path "/d4423042-afac-4db6-85ab-0d70d2d13e98"
+					(reference "FID1")
+					(unit 1)
+				)
+			)
+		)
+	)
+	(symbol
+		(lib_id "Mechanical:Fiducial")
+		(at 162.56 149.86 0)
+		(unit 1)
+		(in_bom no)
+		(on_board yes)
+		(dnp no)
+		(property "Reference" "FID2"
+			(at 162.56 144.78 0)
+			(effects
+				(font
+					(size 1.27 1.27)
+				)
+			)
+		)
+		(property "Value" "Fiducial"
+			(at 162.56 146.685 0)
+			(effects
+				(font
+					(size 1.27 1.27)
+				)
+			)
+		)
+		(property "Footprint" "Fiducial:Fiducial_1mm_Mask2mm"
+			(at 162.56 149.86 0)
+			(hide yes)
+			(effects
+				(font
+					(size 1.27 1.27)
+				)
+			)
+		)
+		(property "LCSC" "C9000033"
+			(at 162.56 149.86 0)
+			(hide yes)
+			(effects
+				(font
+					(size 1.27 1.27)
+				)
+			)
+		)
+		(property "Datasheet" ""
+			(at 162.56 149.86 0)
+			(hide yes)
+			(effects
+				(font
+					(size 1.27 1.27)
+				)
+			)
+		)
+		(property "Description" "Fiducial Marker"
+			(at 162.56 149.86 0)
+			(hide yes)
+			(effects
+				(font
+					(size 1.27 1.27)
+				)
+			)
+		)
+		(instances
+			(project "review-proof"
+				(path "/d4423042-afac-4db6-85ab-0d70d2d13e98"
+					(reference "FID2")
+					(unit 1)
+				)
+			)
+		)
+	)
+	(symbol
+		(lib_id "Mechanical:Fiducial")
+		(at 177.8 149.86 0)
+		(unit 1)
+		(in_bom no)
+		(on_board yes)
+		(dnp no)
+		(property "Reference" "FID3"
+			(at 177.8 144.78 0)
+			(effects
+				(font
+					(size 1.27 1.27)
+				)
+			)
+		)
+		(property "Value" "Fiducial"
+			(at 177.8 146.685 0)
+			(effects
+				(font
+					(size 1.27 1.27)
+				)
+			)
+		)
+		(property "Footprint" "Fiducial:Fiducial_1mm_Mask2mm"
+			(at 177.8 149.86 0)
+			(hide yes)
+			(effects
+				(font
+					(size 1.27 1.27)
+				)
+			)
+		)
+		(property "LCSC" "C9000034"
+			(at 177.8 149.86 0)
+			(hide yes)
+			(effects
+				(font
+					(size 1.27 1.27)
+				)
+			)
+		)
+		(property "Datasheet" ""
+			(at 177.8 149.86 0)
+			(hide yes)
+			(effects
+				(font
+					(size 1.27 1.27)
+				)
+			)
+		)
+		(property "Description" "Fiducial Marker"
+			(at 177.8 149.86 0)
+			(hide yes)
+			(effects
+				(font
+					(size 1.27 1.27)
+				)
+			)
+		)
+		(instances
+			(project "review-proof"
+				(path "/d4423042-afac-4db6-85ab-0d70d2d13e98"
+					(reference "FID3")
+					(unit 1)
+				)
+			)
 		)
 	)
