File: hardware/sunbeam-em7000/main-board/101-mains-entry-and-load-feed.kicad_sch (KiCad schematic)
At the start: 32 parts, among them J101 TAB1_LINE1, J102 TAB2_LINE_IN, J103 TAB3_NEUTRAL_IN, J106 TAB6_COFVALVE, J107 TAB7_COFFPUMP, J108 TAB8_STEAMPUMP, J109 TAB9_HOTVALVE, J110 WB_RET

Commit message: fix(hardware): state the catalogue number none on the hand-fitted symbols, class the 75 V resistors and enable the project's ERC and board checks [SOL-HW-MAIN-BOARD-SCHEMATIC-PROVEN.C2, .C7]
Co-Authored-By: Claude Sonnet 5.5 <noreply@anthropic.com>
Parts:
- JP101, TP101, TP102, TP103, TP104, TP105, TP106, TP107, TP108: LCSC (none) -> none
Changed lines of the file:
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@@
 			)
 		)
-	)
+		(property "LCSC" "none"
+			(at 58.42 40.64 0)
+			(hide yes)
+			(effects
+				(font
+					(size 1.27 1.27)
+				)
+			)
+		))
 	(symbol
 		(lib_id "Device:Fuse")
@@
 			)
 		)
-	)
+		(property "LCSC" "none"
+			(at 119.38 40.64 0)
+			(hide yes)
+			(effects
+				(font
+					(size 1.27 1.27)
+				)
+			)
+		))
 	(symbol
 		(lib_id "Connector_Generic:Conn_01x02")
@@
 			)
 		)
-		(property "LCSC" ""
+		(property "LCSC" "none"
 			(at 149.86 40.64 0)
 			(hide yes)
@@
 			)
 		)
-	)
+		(property "LCSC" "none"
+			(at 180.34 40.64 0)
+			(hide yes)
+			(effects
+				(font
+					(size 1.27 1.27)
+				)
+			)
+		))
 	(symbol
 		(lib_id "Device:Varistor")
@@
 			)
 		)
-	)
+		(property "LCSC" "none"
+			(at 58.42 99.06 0)
+			(hide yes)
+			(effects
+				(font
+					(size 1.27 1.27)
+				)
+			)
+		))
 	(symbol
 		(lib_id "Connector_Generic:Conn_01x01")
@@
 			)
 		)
-	)
+		(property "LCSC" "none"
+			(at 58.42 139.7 0)
+			(hide yes)
+			(effects
+				(font
+					(size 1.27 1.27)
+				)
+			)
+		))
 	(symbol
 		(lib_id "Device:R_Shunt")
@@
 			)
 		)
-	)
+		(property "LCSC" "none"
+			(at 167.64 139.7 0)
+			(hide yes)
+			(effects
+				(font
+					(size 1.27 1.27)
+				)
+			)
+		))
 	(symbol
 		(lib_id "Connector_Generic:Conn_01x01")
@@
 			)
 		)
-	)
+		(property "LCSC" "none"
+			(at 73.66 139.7 0)
+			(hide yes)
+			(effects
+				(font
+					(size 1.27 1.27)
+				)
+			)
+		))
 	(symbol
 		(lib_id "Connector:TestPoint")
@@
 			)
 		)
-	)
+		(property "LCSC" "none"
+			(at 182.88 139.7 0)
+			(hide yes)
+			(effects
+				(font
+					(size 1.27 1.27)
+				)
+			)
+		))
 )

Commit message: fix(hardware): move the symbols with mismatched footprint filters into the board's own library [SOL-HW-MAIN-BOARD-SCHEMATIC-PROVEN.C2, .C7]
Co-Authored-By: Claude Sonnet 5.5 <noreply@anthropic.com>
Parts:
- J101, J102, J103, J106, J107, J108, J109, J110: symbol Connector_Generic:Conn_01x01 -> main-board:Conn_01x01
- JP101: symbol Connector_Generic:Conn_01x02 -> main-board:Conn_01x02
- R105: symbol Device:R_Shunt -> main-board:R_Shunt
Changed lines of the file:
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@@
 	)
 	(symbol
-		(lib_id "Connector_Generic:Conn_01x01")
+		(lib_id "main-board:Conn_01x01")
 		(at 30.48 40.64 0)
 		(unit 1)
@@
 		))
 	(symbol
-		(lib_id "Connector_Generic:Conn_01x02")
+		(lib_id "main-board:Conn_01x02")
 		(at 149.86 40.64 0)
 		(unit 1)
@@
 	)
 	(symbol
-		(lib_id "Connector_Generic:Conn_01x01")
+		(lib_id "main-board:Conn_01x01")
 		(at 30.48 99.06 0)
 		(unit 1)
@@
 		))
 	(symbol
-		(lib_id "Connector_Generic:Conn_01x01")
+		(lib_id "main-board:Conn_01x01")
 		(at 30.48 139.7 0)
 		(unit 1)
@@
 		))
 	(symbol
-		(lib_id "Device:R_Shunt")
+		(lib_id "main-board:R_Shunt")
 		(at 99.06 139.7 0)
 		(unit 1)
@@
 	)
 	(symbol
-		(lib_id "Connector_Generic:Conn_01x01")
+		(lib_id "main-board:Conn_01x01")
 		(at 139.7 139.7 0)
 		(unit 1)
@@
 		))
 	(symbol
-		(lib_id "Connector_Generic:Conn_01x01")
+		(lib_id "main-board:Conn_01x01")
 		(at 220.98 119.38 0)
 		(unit 1)
@@
 	)
 	(symbol
-		(lib_id "Connector_Generic:Conn_01x01")
+		(lib_id "main-board:Conn_01x01")
 		(at 220.98 139.7 0)
 		(unit 1)
@@
 	)
 	(symbol
-		(lib_id "Connector_Generic:Conn_01x01")
+		(lib_id "main-board:Conn_01x01")
 		(at 220.98 160.02 0)
 		(unit 1)
@@
 	)
 	(symbol
-		(lib_id "Connector_Generic:Conn_01x01")
+		(lib_id "main-board:Conn_01x01")
 		(at 220.98 180.34 0)
 		(unit 1)

Commit message: main-board: point the 96 test-point symbols and Y601 at the small test-point and marked oscillator footprints [SOL-HW-MAIN-BOARD-PROVEN-AND-LAID-OUT.C8]
Co-Authored-By: Claude Sonnet 5.5 <noreply@anthropic.com>
Parts:
- TP101, TP102, TP103, TP104, TP105, TP106, TP107, TP108: footprint TestPoint:TestPoint_Pad_D1.5mm -> main-board:TestPoint_Pad_D1.0mm_Tight
Changed lines of the file:
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@@
 			)
 		)
-		(property "Footprint" "TestPoint:TestPoint_Pad_D1.5mm"
+		(property "Footprint" "main-board:TestPoint_Pad_D1.0mm_Tight"
 			(at 58.42 40.64 0)
 			(hide yes)
@@
 			)
 		)
-		(property "Footprint" "TestPoint:TestPoint_Pad_D1.5mm"
+		(property "Footprint" "main-board:TestPoint_Pad_D1.0mm_Tight"
 			(at 119.38 40.64 0)
 			(hide yes)
@@
 			)
 		)
-		(property "Footprint" "TestPoint:TestPoint_Pad_D1.5mm"
+		(property "Footprint" "main-board:TestPoint_Pad_D1.0mm_Tight"
 			(at 180.34 40.64 0)
 			(hide yes)
@@
 			)
 		)
-		(property "Footprint" "TestPoint:TestPoint_Pad_D1.5mm"
+		(property "Footprint" "main-board:TestPoint_Pad_D1.0mm_Tight"
 			(at 58.42 99.06 0)
 			(hide yes)
@@
 			)
 		)
-		(property "Footprint" "TestPoint:TestPoint_Pad_D1.5mm"
+		(property "Footprint" "main-board:TestPoint_Pad_D1.0mm_Tight"
 			(at 58.42 139.7 0)
 			(hide yes)
@@
 			)
 		)
-		(property "Footprint" "TestPoint:TestPoint_Pad_D1.5mm"
+		(property "Footprint" "main-board:TestPoint_Pad_D1.0mm_Tight"
 			(at 167.64 139.7 0)
 			(hide yes)
@@
 			)
 		)
-		(property "Footprint" "TestPoint:TestPoint_Pad_D1.5mm"
+		(property "Footprint" "main-board:TestPoint_Pad_D1.0mm_Tight"
 			(at 73.66 139.7 0)
 			(hide yes)
@@
 			)
 		)
-		(property "Footprint" "TestPoint:TestPoint_Pad_D1.5mm"
+		(property "Footprint" "main-board:TestPoint_Pad_D1.0mm_Tight"
 			(at 182.88 139.7 0)
 			(hide yes)
