File: hardware/sunbeam-em7000/main-board/52-flow-pressure-and-spare-analogue-inputs.kicad_sch (KiCad schematic)
At the start: 67 parts, among them J520 FLOW, J521 STM_D, J522 BREW_D, J523 SPARE_A, J524 BREW_A, J525 SPARE_AN2_H, U520 SN74LVC1G17

Commit message: fix(hardware): state the catalogue number none on the hand-fitted symbols, class the 75 V resistors and enable the project's ERC and board checks [SOL-HW-MAIN-BOARD-SCHEMATIC-PROVEN.C2, .C7]
Co-Authored-By: Claude Sonnet 5.5 <noreply@anthropic.com>
Parts:
- TP520, TP521, TP522, TP523, TP524, TP525, TP526, TP527, TP528, TP529, TP530, TP531, TP532: LCSC (none) -> none
Changed lines of the file:
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@@
 				)
 			)
+		)
+		(property "LCSC" "none"
+			(at 167.64 50.8 0)
+			(hide yes)
+			(effects
+				(font
+					(size 1.27 1.27)
+				)
+			)
 		))
 	(symbol
@@
 				)
 			)
+		)
+		(property "LCSC" "none"
+			(at 116.84 111.76 0)
+			(hide yes)
+			(effects
+				(font
+					(size 1.27 1.27)
+				)
+			)
 		))
 	(symbol
@@
 				)
 			)
+		)
+		(property "LCSC" "none"
+			(at 167.64 147.32 0)
+			(hide yes)
+			(effects
+				(font
+					(size 1.27 1.27)
+				)
+			)
 		))
 	(symbol
@@
 				)
 			)
+		)
+		(property "LCSC" "none"
+			(at 167.64 182.88 0)
+			(hide yes)
+			(effects
+				(font
+					(size 1.27 1.27)
+				)
+			)
 		))
 	(symbol
@@
 				)
 			)
+		)
+		(property "LCSC" "none"
+			(at 116.84 222.25 0)
+			(hide yes)
+			(effects
+				(font
+					(size 1.27 1.27)
+				)
+			)
 		))
 	(symbol
@@
 				)
 			)
+		)
+		(property "LCSC" "none"
+			(at 167.64 257.81 0)
+			(hide yes)
+			(effects
+				(font
+					(size 1.27 1.27)
+				)
+			)
 		))
 	(symbol
@@
 				)
 			)
+		)
+		(property "LCSC" "none"
+			(at 167.64 293.37 0)
+			(hide yes)
+			(effects
+				(font
+					(size 1.27 1.27)
+				)
+			)
 		))
 	(symbol
@@
 				)
 			)
+		)
+		(property "LCSC" "none"
+			(at 330.2 50.8 0)
+			(hide yes)
+			(effects
+				(font
+					(size 1.27 1.27)
+				)
+			)
 		))
 	(symbol
@@
 				)
 			)
+		)
+		(property "LCSC" "none"
+			(at 406.4 88.9 0)
+			(hide yes)
+			(effects
+				(font
+					(size 1.27 1.27)
+				)
+			)
 		))
 	(symbol
@@
 				)
 			)
+		)
+		(property "LCSC" "none"
+			(at 330.2 152.4 0)
+			(hide yes)
+			(effects
+				(font
+					(size 1.27 1.27)
+				)
+			)
 		))
 	(symbol
@@
 				)
 			)
+		)
+		(property "LCSC" "none"
+			(at 406.4 190.5 0)
+			(hide yes)
+			(effects
+				(font
+					(size 1.27 1.27)
+				)
+			)
 		))
 	(symbol
@@
 				)
 			)
+		)
+		(property "LCSC" "none"
+			(at 330.2 254 0)
+			(hide yes)
+			(effects
+				(font
+					(size 1.27 1.27)
+				)
+			)
 		))
 	(symbol
@@
 			(at 406.4 292.1 0)
 			(hide yes)
+			(effects
+				(font
+					(size 1.27 1.27)
+				)
+			)
+		)
+		(property "LCSC" "none"
+			(at 406.4 292.1 0)
+			(hide yes)

Commit message: fix(hardware): move the symbols with mismatched footprint filters into the board's own library [SOL-HW-MAIN-BOARD-SCHEMATIC-PROVEN.C2, .C7]
Co-Authored-By: Claude Sonnet 5.5 <noreply@anthropic.com>
Parts:
- F520, F521, F522, F523, F524: symbol Device:Polyfuse -> main-board:Polyfuse
- U520: symbol 74xGxx:74LVC1G17 -> main-board:74LVC1G17
Changed lines of the file:
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@@
 		))
 	(symbol
-		(lib_id "74xGxx:74LVC1G17")
+		(lib_id "main-board:74LVC1G17")
 		(at 142.24 76.2 0)
 		(unit 1)
@@
 		))
 	(symbol
-		(lib_id "Device:Polyfuse")
+		(lib_id "main-board:Polyfuse")
 		(at 66.04 111.76 0)
 		(unit 1)
@@
 		))
 	(symbol
-		(lib_id "Device:Polyfuse")
+		(lib_id "main-board:Polyfuse")
 		(at 66.04 222.25 0)
 		(unit 1)
@@
 		))
 	(symbol
-		(lib_id "Device:Polyfuse")
+		(lib_id "main-board:Polyfuse")
 		(at 279.4 50.8 0)
 		(unit 1)
@@
 		))
 	(symbol
-		(lib_id "Device:Polyfuse")
+		(lib_id "main-board:Polyfuse")
 		(at 279.4 152.4 0)
 		(unit 1)
@@
 		))
 	(symbol
-		(lib_id "Device:Polyfuse")
+		(lib_id "main-board:Polyfuse")
 		(at 279.4 254 0)
 		(unit 1)

Commit message: main-board: point the 96 test-point symbols and Y601 at the small test-point and marked oscillator footprints [SOL-HW-MAIN-BOARD-PROVEN-AND-LAID-OUT.C8]
Co-Authored-By: Claude Sonnet 5.5 <noreply@anthropic.com>
Parts:
- TP520, TP521, TP522, TP523, TP524, TP525, TP526, TP527, TP528, TP529, TP530, TP531, TP532: footprint TestPoint:TestPoint_Pad_D1.5mm -> main-board:TestPoint_Pad_D1.0mm_Tight
Changed lines of the file:
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@@
 			)
 		)
-		(property "Footprint" "TestPoint:TestPoint_Pad_D1.5mm"
+		(property "Footprint" "main-board:TestPoint_Pad_D1.0mm_Tight"
 			(at 167.64 50.8 0)
 			(hide yes)
@@
 			)
 		)
-		(property "Footprint" "TestPoint:TestPoint_Pad_D1.5mm"
+		(property "Footprint" "main-board:TestPoint_Pad_D1.0mm_Tight"
 			(at 116.84 111.76 0)
 			(hide yes)
@@
 			)
 		)
-		(property "Footprint" "TestPoint:TestPoint_Pad_D1.5mm"
+		(property "Footprint" "main-board:TestPoint_Pad_D1.0mm_Tight"
 			(at 167.64 147.32 0)
 			(hide yes)
@@
 			)
 		)
-		(property "Footprint" "TestPoint:TestPoint_Pad_D1.5mm"
+		(property "Footprint" "main-board:TestPoint_Pad_D1.0mm_Tight"
 			(at 167.64 182.88 0)
 			(hide yes)
@@
 			)
 		)
-		(property "Footprint" "TestPoint:TestPoint_Pad_D1.5mm"
+		(property "Footprint" "main-board:TestPoint_Pad_D1.0mm_Tight"
 			(at 116.84 222.25 0)
 			(hide yes)
@@
 			)
 		)
-		(property "Footprint" "TestPoint:TestPoint_Pad_D1.5mm"
+		(property "Footprint" "main-board:TestPoint_Pad_D1.0mm_Tight"
 			(at 167.64 257.81 0)
 			(hide yes)
@@
 			)
 		)
-		(property "Footprint" "TestPoint:TestPoint_Pad_D1.5mm"
+		(property "Footprint" "main-board:TestPoint_Pad_D1.0mm_Tight"
 			(at 167.64 293.37 0)
 			(hide yes)
@@
 			)
 		)
-		(property "Footprint" "TestPoint:TestPoint_Pad_D1.5mm"
+		(property "Footprint" "main-board:TestPoint_Pad_D1.0mm_Tight"
 			(at 330.2 50.8 0)
 			(hide yes)
@@
 			)
 		)
-		(property "Footprint" "TestPoint:TestPoint_Pad_D1.5mm"
+		(property "Footprint" "main-board:TestPoint_Pad_D1.0mm_Tight"
 			(at 406.4 88.9 0)
 			(hide yes)
@@
 			)
 		)
-		(property "Footprint" "TestPoint:TestPoint_Pad_D1.5mm"
+		(property "Footprint" "main-board:TestPoint_Pad_D1.0mm_Tight"
 			(at 330.2 152.4 0)
 			(hide yes)
@@
 			)
 		)
-		(property "Footprint" "TestPoint:TestPoint_Pad_D1.5mm"
+		(property "Footprint" "main-board:TestPoint_Pad_D1.0mm_Tight"
 			(at 406.4 190.5 0)
 			(hide yes)
@@
 			)
 		)
-		(property "Footprint" "TestPoint:TestPoint_Pad_D1.5mm"
+		(property "Footprint" "main-board:TestPoint_Pad_D1.0mm_Tight"
 			(at 330.2 254 0)
 			(hide yes)
@@
 			)
 		)
-		(property "Footprint" "TestPoint:TestPoint_Pad_D1.5mm"
+		(property "Footprint" "main-board:TestPoint_Pad_D1.0mm_Tight"
 			(at 406.4 292.1 0)
 			(hide yes)
