File: hardware/sunbeam-em7000/main-board/710-valve-drives.kicad_sch (KiCad schematic)
At the start: 13 parts, among them K731 HF32FA-G/005-HSL1, K741 HF32FA-G/005-HSL1, Q731 AO3400A, Q741 AO3400A

Commit message: fix(hardware): state the catalogue number none on the hand-fitted symbols, class the 75 V resistors and enable the project's ERC and board checks [SOL-HW-MAIN-BOARD-SCHEMATIC-PROVEN.C2, .C7]
Co-Authored-By: Claude Sonnet 5.5 <noreply@anthropic.com>
Parts:
- TP731, TP741: LCSC (none) -> none
Changed lines of the file:
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@@
 			)
 		)
-		(property "LCSC" ""
+		(property "LCSC" "none"
 			(at 104.14 91.44 0)
 			(hide yes)
@@
 			)
 		)
-		(property "LCSC" ""
+		(property "LCSC" "none"
 			(at 104.14 182.88 0)
 			(hide yes)

Commit message: fix(hardware): move the symbols with mismatched footprint filters into the board's own library [SOL-HW-MAIN-BOARD-SCHEMATIC-PROVEN.C2, .C7]
Co-Authored-By: Claude Sonnet 5.5 <noreply@anthropic.com>
Parts:
- K731, K741: symbol Relay:Relay_SPST-NO -> main-board:Relay_SPST-NO
Changed lines of the file:
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@@
 		))
 	(symbol
-		(lib_id "Relay:Relay_SPST-NO")
+		(lib_id "main-board:Relay_SPST-NO")
 		(at 152.4 60.96 0)
 		(mirror y)
@@
 		))
 	(symbol
-		(lib_id "Relay:Relay_SPST-NO")
+		(lib_id "main-board:Relay_SPST-NO")
 		(at 152.4 152.4 0)
 		(mirror y)

Commit message: main-board: point the 96 test-point symbols and Y601 at the small test-point and marked oscillator footprints [SOL-HW-MAIN-BOARD-PROVEN-AND-LAID-OUT.C8]
Co-Authored-By: Claude Sonnet 5.5 <noreply@anthropic.com>
Parts:
- TP731, TP741: footprint TestPoint:TestPoint_Pad_D1.5mm -> main-board:TestPoint_Pad_D1.0mm_Tight
Changed lines of the file:
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@@
 			)
 		)
-		(property "Footprint" "TestPoint:TestPoint_Pad_D1.5mm"
+		(property "Footprint" "main-board:TestPoint_Pad_D1.0mm_Tight"
 			(at 104.14 91.44 0)
 			(hide yes)
@@
 			)
 		)
-		(property "Footprint" "TestPoint:TestPoint_Pad_D1.5mm"
+		(property "Footprint" "main-board:TestPoint_Pad_D1.0mm_Tight"
 			(at 104.14 182.88 0)
 			(hide yes)
