File: hardware/sunbeam-em7000/main-board/720-heater-led-drive-and-wall-board-header.kicad_sch (KiCad schematic)
At the start: 17 parts, among them J761 WB_LV10, Q761 AO3400A, Q771 AO3400A

Commit message: fix(hardware): state the catalogue number none on the hand-fitted symbols, class the 75 V resistors and enable the project's ERC and board checks [SOL-HW-MAIN-BOARD-SCHEMATIC-PROVEN.C2, .C7]
Co-Authored-By: Claude Sonnet 5.5 <noreply@anthropic.com>
Parts:
- TP761, TP762, TP772: LCSC (none) -> none
Changed lines of the file:
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@@
 			)
 		)
-	)
+		(property "LCSC" "none"
+			(at 50.8 40.64 0)
+			(hide yes)
+			(effects
+				(font
+					(size 1.27 1.27)
+				)
+			)
+		))
 	(symbol
 		(lib_id "Device:R")
@@
 			)
 		)
-	)
+		(property "LCSC" "none"
+			(at 50.8 91.44 0)
+			(hide yes)
+			(effects
+				(font
+					(size 1.27 1.27)
+				)
+			)
+		))
 	(symbol
 		(lib_id "Connector_Generic:Conn_01x10")
@@
 			)
 		)
-	)
+		(property "LCSC" "none"
+			(at 227.33 152.4 0)
+			(hide yes)
+			(effects
+				(font
+					(size 1.27 1.27)
+				)
+			)
+		))
 	(symbol
 		(lib_id "power:GND")

Commit message: main-board: point the 96 test-point symbols and Y601 at the small test-point and marked oscillator footprints [SOL-HW-MAIN-BOARD-PROVEN-AND-LAID-OUT.C8]
Co-Authored-By: Claude Sonnet 5.5 <noreply@anthropic.com>
Parts:
- TP761, TP762, TP772: footprint TestPoint:TestPoint_Pad_D1.5mm -> main-board:TestPoint_Pad_D1.0mm_Tight
Changed lines of the file:
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@@
 			)
 		)
-		(property "Footprint" "TestPoint:TestPoint_Pad_D1.5mm"
+		(property "Footprint" "main-board:TestPoint_Pad_D1.0mm_Tight"
 			(at 50.8 40.64 0)
 			(hide yes)
@@
 			)
 		)
-		(property "Footprint" "TestPoint:TestPoint_Pad_D1.5mm"
+		(property "Footprint" "main-board:TestPoint_Pad_D1.0mm_Tight"
 			(at 50.8 91.44 0)
 			(hide yes)
@@
 			)
 		)
-		(property "Footprint" "TestPoint:TestPoint_Pad_D1.5mm"
+		(property "Footprint" "main-board:TestPoint_Pad_D1.0mm_Tight"
 			(at 227.33 152.4 0)
 			(hide yes)
