File: hardware/sunbeam-em7000/main-board/E2-zero-crossing-detector.kicad_sch (KiCad schematic)
At the start: 6 parts, among them U602 LTV-814S-TA1-A

Commit message: fix(hardware): state the catalogue number none on the hand-fitted symbols, class the 75 V resistors and enable the project's ERC and board checks [SOL-HW-MAIN-BOARD-SCHEMATIC-PROVEN.C2, .C7]
Co-Authored-By: Claude Sonnet 5.5 <noreply@anthropic.com>
Parts:
- TP630: LCSC (none) -> none
Changed lines of the file:
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@@
 			)
 		)
-	)
+		(property "LCSC" "none"
+			(at 121.92 77.47 0)
+			(hide yes)
+			(effects
+				(font
+					(size 1.27 1.27)
+				)
+			)
+		))
 	(symbol
 		(lib_id "power:+3V3")

Commit message: main-board: point the 96 test-point symbols and Y601 at the small test-point and marked oscillator footprints [SOL-HW-MAIN-BOARD-PROVEN-AND-LAID-OUT.C8]
Co-Authored-By: Claude Sonnet 5.5 <noreply@anthropic.com>
Parts:
- TP630: footprint TestPoint:TestPoint_Pad_D1.5mm -> main-board:TestPoint_Pad_D1.0mm_Tight
Changed lines of the file:
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@@
 			)
 		)
-		(property "Footprint" "TestPoint:TestPoint_Pad_D1.5mm"
+		(property "Footprint" "main-board:TestPoint_Pad_D1.0mm_Tight"
 			(at 121.92 77.47 0)
 			(hide yes)
