File: hardware/sunbeam-em7000/main-board/E4-load-cell-amplifiers.kicad_sch (KiCad schematic)
At the start: 22 parts, among them J630 WT1_H, J635 WT2_H, U630 HX711, U631 HX711

Commit message: fix(hardware): state the catalogue number none on the hand-fitted symbols, class the 75 V resistors and enable the project's ERC and board checks [SOL-HW-MAIN-BOARD-SCHEMATIC-PROVEN.C2, .C7]
Co-Authored-By: Claude Sonnet 5.5 <noreply@anthropic.com>
Parts:
- TP670, TP671, TP672, TP673: LCSC (none) -> none
Changed lines of the file:
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@@
 			)
 		)
-	)
+		(property "LCSC" "none"
+			(at 190.5 68.58 0)
+			(hide yes)
+			(effects
+				(font
+					(size 1.27 1.27)
+				)
+			)
+		))
 	(symbol
 		(lib_id "Connector:TestPoint")
@@
 			)
 		)
-	)
+		(property "LCSC" "none"
+			(at 124.46 71.12 0)
+			(hide yes)
+			(effects
+				(font
+					(size 1.27 1.27)
+				)
+			)
+		))
 	(symbol
 		(lib_id "Analog_ADC:HX711")
@@
 			)
 		)
-	)
+		(property "LCSC" "none"
+			(at 190.5 170.18 0)
+			(hide yes)
+			(effects
+				(font
+					(size 1.27 1.27)
+				)
+			)
+		))
 	(symbol
 		(lib_id "Connector:TestPoint")
@@
 			)
 		)
-	)
+		(property "LCSC" "none"
+			(at 124.46 172.72 0)
+			(hide yes)
+			(effects
+				(font
+					(size 1.27 1.27)
+				)
+			)
+		))
 	(symbol
 		(lib_id "power:+5V")

Commit message: main-board: point the 96 test-point symbols and Y601 at the small test-point and marked oscillator footprints [SOL-HW-MAIN-BOARD-PROVEN-AND-LAID-OUT.C8]
Co-Authored-By: Claude Sonnet 5.5 <noreply@anthropic.com>
Parts:
- TP670, TP671, TP672, TP673: footprint TestPoint:TestPoint_Pad_D1.5mm -> main-board:TestPoint_Pad_D1.0mm_Tight
Changed lines of the file:
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@@
 			)
 		)
-		(property "Footprint" "TestPoint:TestPoint_Pad_D1.5mm"
+		(property "Footprint" "main-board:TestPoint_Pad_D1.0mm_Tight"
 			(at 190.5 68.58 0)
 			(hide yes)
@@
 			)
 		)
-		(property "Footprint" "TestPoint:TestPoint_Pad_D1.5mm"
+		(property "Footprint" "main-board:TestPoint_Pad_D1.0mm_Tight"
 			(at 124.46 71.12 0)
 			(hide yes)
@@
 			)
 		)
-		(property "Footprint" "TestPoint:TestPoint_Pad_D1.5mm"
+		(property "Footprint" "main-board:TestPoint_Pad_D1.0mm_Tight"
 			(at 190.5 170.18 0)
 			(hide yes)
@@
 			)
 		)
-		(property "Footprint" "TestPoint:TestPoint_Pad_D1.5mm"
+		(property "Footprint" "main-board:TestPoint_Pad_D1.0mm_Tight"
 			(at 124.46 172.72 0)
 			(hide yes)
