File: hardware/sunbeam-em7000/main-board/700-pump-drives.kicad_sch (KiCad schematic)
At the start: 26 parts, among them Q701 AO3400A, Q711 AO3400A, T701 BTA204S-600B, T711 BTA204S-600B, U701 MOC3052SVM, U711 MOC3052SVM

Commit message: fix(hardware): state the catalogue number none on the hand-fitted symbols, class the 75 V resistors and enable the project's ERC and board checks [SOL-HW-MAIN-BOARD-SCHEMATIC-PROVEN.C2, .C7]
Co-Authored-By: Claude Sonnet 5.5 <noreply@anthropic.com>
Parts:
- TP701, TP702, TP711, TP712: LCSC (none) -> none
Changed lines of the file:
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@@
 			)
 		)
-		(property "LCSC" ""
+		(property "LCSC" "none"
 			(at 35.56 49.53 0)
 			(hide yes)
@@
 			)
 		)
-		(property "LCSC" ""
+		(property "LCSC" "none"
 			(at 35.56 139.7 0)
 			(hide yes)
@@
 			)
 		)
-		(property "LCSC" ""
+		(property "LCSC" "none"
 			(at 233.68 60.96 0)
 			(hide yes)
@@
 			)
 		)
-		(property "LCSC" ""
+		(property "LCSC" "none"
 			(at 233.68 151.13 0)
 			(hide yes)

Commit message: fix(hardware): move the symbols with mismatched footprint filters into the board's own library [SOL-HW-MAIN-BOARD-SCHEMATIC-PROVEN.C2, .C7]
Co-Authored-By: Claude Sonnet 5.5 <noreply@anthropic.com>
Parts:
- T701, T711: symbol Triac_Thyristor:BT136-600 -> main-board:BT136-600
- U701, U711: symbol Relay_SolidState:MOC3052M -> main-board:MOC3052M
Changed lines of the file:
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@@
 		))
 	(symbol
-		(lib_id "Relay_SolidState:MOC3052M")
+		(lib_id "main-board:MOC3052M")
 		(at 149.86 64.77 0)
 		(unit 1)
@@
 		))
 	(symbol
-		(lib_id "Triac_Thyristor:BT136-600")
+		(lib_id "main-board:BT136-600")
 		(at 214.63 69.85 0)
 		(unit 1)
@@
 		))
 	(symbol
-		(lib_id "Relay_SolidState:MOC3052M")
+		(lib_id "main-board:MOC3052M")
 		(at 149.86 154.94 0)
 		(unit 1)
@@
 		))
 	(symbol
-		(lib_id "Triac_Thyristor:BT136-600")
+		(lib_id "main-board:BT136-600")
 		(at 214.63 160.02 0)
 		(unit 1)

Commit message: main-board: point the 96 test-point symbols and Y601 at the small test-point and marked oscillator footprints [SOL-HW-MAIN-BOARD-PROVEN-AND-LAID-OUT.C8]
Co-Authored-By: Claude Sonnet 5.5 <noreply@anthropic.com>
Parts:
- TP701, TP702, TP711, TP712: footprint TestPoint:TestPoint_Pad_D1.5mm -> main-board:TestPoint_Pad_D1.0mm_Tight
Changed lines of the file:
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@@
 			)
 		)
-		(property "Footprint" "TestPoint:TestPoint_Pad_D1.5mm"
+		(property "Footprint" "main-board:TestPoint_Pad_D1.0mm_Tight"
 			(at 35.56 49.53 0)
 			(hide yes)
@@
 			)
 		)
-		(property "Footprint" "TestPoint:TestPoint_Pad_D1.5mm"
+		(property "Footprint" "main-board:TestPoint_Pad_D1.0mm_Tight"
 			(at 35.56 139.7 0)
 			(hide yes)
@@
 			)
 		)
-		(property "Footprint" "TestPoint:TestPoint_Pad_D1.5mm"
+		(property "Footprint" "main-board:TestPoint_Pad_D1.0mm_Tight"
 			(at 233.68 60.96 0)
 			(hide yes)
@@
 			)
 		)
-		(property "Footprint" "TestPoint:TestPoint_Pad_D1.5mm"
+		(property "Footprint" "main-board:TestPoint_Pad_D1.0mm_Tight"
 			(at 233.68 151.13 0)
 			(hide yes)

Commit message: feat(hardware): fit the pump triacs with the two-lead tab land [SOL-HW-MAIN-BOARD-PROVEN-AND-LAID-OUT.C18]
Co-Authored-By: Claude Sonnet 5.5 <noreply@anthropic.com>
Parts:
- T701, T711: footprint Package_TO_SOT_SMD:TO-252-3_TabPin2 -> main-board:TO-252-2_TabPin2_Triac
Changed lines of the file:
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@@
 			)
 		)
-		(property "Footprint" "Package_TO_SOT_SMD:TO-252-3_TabPin2"
+		(property "Footprint" "main-board:TO-252-2_TabPin2_Triac"
 			(at 214.63 69.85 0)
 			(hide yes)
@@
 			)
 		)
-		(property "Footprint" "Package_TO_SOT_SMD:TO-252-3_TabPin2"
+		(property "Footprint" "main-board:TO-252-2_TabPin2_Triac"
 			(at 214.63 160.02 0)
 			(hide yes)
