File: hardware/sunbeam-em7000/main-board/E1-supply-voltage-and-current-measurement.kicad_sch (KiCad schematic)
At the start: 41 parts, among them U601 AMC131M02, Y601 8.000MHz

Commit message: fix(hardware): state the catalogue number none on the hand-fitted symbols, class the 75 V resistors and enable the project's ERC and board checks [SOL-HW-MAIN-BOARD-SCHEMATIC-PROVEN.C2, .C7]
Co-Authored-By: Claude Sonnet 5.5 <noreply@anthropic.com>
Parts:
- TP601, TP602, TP603, TP604, TP605, TP606, TP607, TP608, TP609, TP610: LCSC (none) -> none
Changed lines of the file:
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@@
 			)
 		)
-	)
+		(property "LCSC" "none"
+			(at 80.01 68.58 0)
+			(hide yes)
+			(effects
+				(font
+					(size 1.27 1.27)
+				)
+			)
+		))
 	(symbol
 		(lib_id "Connector:TestPoint")
@@
 			)
 		)
-	)
+		(property "LCSC" "none"
+			(at 69.85 114.3 0)
+			(hide yes)
+			(effects
+				(font
+					(size 1.27 1.27)
+				)
+			)
+		))
 	(symbol
 		(lib_id "Connector:TestPoint")
@@
 			)
 		)
-	)
+		(property "LCSC" "none"
+			(at 297.18 185.42 0)
+			(hide yes)
+			(effects
+				(font
+					(size 1.27 1.27)
+				)
+			)
+		))
 	(symbol
 		(lib_id "Connector:TestPoint")
@@
 			)
 		)
-	)
+		(property "LCSC" "none"
+			(at 297.18 193.04 0)
+			(hide yes)
+			(effects
+				(font
+					(size 1.27 1.27)
+				)
+			)
+		))
 	(symbol
 		(lib_id "Connector:TestPoint")
@@
 			)
 		)
-	)
+		(property "LCSC" "none"
+			(at 297.18 200.66 0)
+			(hide yes)
+			(effects
+				(font
+					(size 1.27 1.27)
+				)
+			)
+		))
 	(symbol
 		(lib_id "Connector:TestPoint")
@@
 			)
 		)
-	)
+		(property "LCSC" "none"
+			(at 297.18 208.28 0)
+			(hide yes)
+			(effects
+				(font
+					(size 1.27 1.27)
+				)
+			)
+		))
 	(symbol
 		(lib_id "Connector:TestPoint")
@@
 			)
 		)
-	)
+		(property "LCSC" "none"
+			(at 200.66 85.09 0)
+			(hide yes)
+			(effects
+				(font
+					(size 1.27 1.27)
+				)
+			)
+		))
 	(symbol
 		(lib_id "Connector:TestPoint")
@@
 			)
 		)
-	)
+		(property "LCSC" "none"
+			(at 200.66 92.71 0)
+			(hide yes)
+			(effects
+				(font
+					(size 1.27 1.27)
+				)
+			)
+		))
 	(symbol
 		(lib_id "Connector:TestPoint")
@@
 			)
 		)
-	)
+		(property "LCSC" "none"
+			(at 200.66 100.33 0)
+			(hide yes)
+			(effects
+				(font
+					(size 1.27 1.27)
+				)
+			)
+		))
 	(symbol
 		(lib_id "Connector:TestPoint")
@@
 			)
 		)
-	)
+		(property "LCSC" "none"
+			(at 200.66 107.95 0)
+			(hide yes)
+			(effects
+				(font
+					(size 1.27 1.27)
+				)
+			)
+		))
 	(symbol
 		(lib_id "power:+3V3")

Commit message: main-board: point the 96 test-point symbols and Y601 at the small test-point and marked oscillator footprints [SOL-HW-MAIN-BOARD-PROVEN-AND-LAID-OUT.C8]
Co-Authored-By: Claude Sonnet 5.5 <noreply@anthropic.com>
Parts:
- TP601, TP602, TP603, TP604, TP605, TP606, TP607, TP608, TP609, TP610: footprint TestPoint:TestPoint_Pad_D1.5mm -> main-board:TestPoint_Pad_D1.0mm_Tight
- Y601: footprint Oscillator:Oscillator_SMD_Abracon_ASE-4Pin_3.2x2.5mm -> main-board:Oscillator_SMD_Abracon_ASE-4Pin_3.2x2.5mm_Pin1Mark
Changed lines of the file:
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@@
 			)
 		)
-		(property "Footprint" "Oscillator:Oscillator_SMD_Abracon_ASE-4Pin_3.2x2.5mm"
+		(property "Footprint" "main-board:Oscillator_SMD_Abracon_ASE-4Pin_3.2x2.5mm_Pin1Mark"
 			(at 360.68 137.16 0)
 			(hide yes)
@@
 			)
 		)
-		(property "Footprint" "TestPoint:TestPoint_Pad_D1.5mm"
+		(property "Footprint" "main-board:TestPoint_Pad_D1.0mm_Tight"
 			(at 80.01 68.58 0)
 			(hide yes)
@@
 			)
 		)
-		(property "Footprint" "TestPoint:TestPoint_Pad_D1.5mm"
+		(property "Footprint" "main-board:TestPoint_Pad_D1.0mm_Tight"
 			(at 69.85 114.3 0)
 			(hide yes)
@@
 			)
 		)
-		(property "Footprint" "TestPoint:TestPoint_Pad_D1.5mm"
+		(property "Footprint" "main-board:TestPoint_Pad_D1.0mm_Tight"
 			(at 297.18 185.42 0)
 			(hide yes)
@@
 			)
 		)
-		(property "Footprint" "TestPoint:TestPoint_Pad_D1.5mm"
+		(property "Footprint" "main-board:TestPoint_Pad_D1.0mm_Tight"
 			(at 297.18 193.04 0)
 			(hide yes)
@@
 			)
 		)
-		(property "Footprint" "TestPoint:TestPoint_Pad_D1.5mm"
+		(property "Footprint" "main-board:TestPoint_Pad_D1.0mm_Tight"
 			(at 297.18 200.66 0)
 			(hide yes)
@@
 			)
 		)
-		(property "Footprint" "TestPoint:TestPoint_Pad_D1.5mm"
+		(property "Footprint" "main-board:TestPoint_Pad_D1.0mm_Tight"
 			(at 297.18 208.28 0)
 			(hide yes)
@@
 			)
 		)
-		(property "Footprint" "TestPoint:TestPoint_Pad_D1.5mm"
+		(property "Footprint" "main-board:TestPoint_Pad_D1.0mm_Tight"
 			(at 200.66 85.09 0)
 			(hide yes)
@@
 			)
 		)
-		(property "Footprint" "TestPoint:TestPoint_Pad_D1.5mm"
+		(property "Footprint" "main-board:TestPoint_Pad_D1.0mm_Tight"
 			(at 200.66 92.71 0)
 			(hide yes)
@@
 			)
 		)
-		(property "Footprint" "TestPoint:TestPoint_Pad_D1.5mm"
+		(property "Footprint" "main-board:TestPoint_Pad_D1.0mm_Tight"
 			(at 200.66 100.33 0)
 			(hide yes)
@@
 			)
 		)
-		(property "Footprint" "TestPoint:TestPoint_Pad_D1.5mm"
+		(property "Footprint" "main-board:TestPoint_Pad_D1.0mm_Tight"
 			(at 200.66 107.95 0)
 			(hide yes)

Commit message: main-board: split the AMC high-side ground from NEUTRAL at one net tie by the shunt [SOL-HW-MAIN-BOARD-PROVEN-AND-LAID-OUT.C1]
Co-Authored-By: Claude Sonnet 5.5 <noreply@anthropic.com>
Parts:
- added NT601: NetTie_2, NetTie:NetTie-2_SMD_Pad0.5mm, symbol Device:NetTie_2
Connections:
- net NEUTRAL: now also NT601.1; no longer C605.2, C606.2, C607.2, C608.2, F602.2, R604.2, R606.2, U601.5 (HGND)
- new net AMC_HGND: C605.2, C606.2, C607.2, C608.2, F602.2, NT601.2, R604.2, R606.2, U601.5 (HGND)

Commit message: main-board: give the net tie NT601 the LCSC field every part record carries [SOL-HW-MAIN-BOARD-PROVEN-AND-LAID-OUT.C1]
Co-Authored-By: Claude Sonnet 5.5 <noreply@anthropic.com>
Parts:
- NT601: LCSC (none) -> none
Changed lines of the file:
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@@
 			)
 		)
-	)
+		(property "LCSC" "none"
+			(at 71.12 92.71 0)
+			(hide yes)
+			(effects
+				(font
+					(size 1.27 1.27)
+				)
+			)
+		))
 )
